File: cafereg2.brd (EAGLE design)
At the start: 37.4 x 23 mm, 83 parts, among them IC1 SIC431AED-T1-GE3, IC2 MUN3CAD01-SB, IC3 SIC431AED-T1-GE3, IC4 MUN3CAD01-SB, IC5 FAN48610BUC50X

Commit message: update bom
Parts:
- removed C56: 22uF, resistor:C0603
- removed PS1: TPS63810YFFR, SamacSys_Parts:BGA15C40P3X5_134X226X62
- removed PS2: MUN3CAD03-SE, SamacSys_Parts:MUN3CAD03SE
- removed R19: 11k, resistor:R0402
- removed R20: 12k, resistor:R0402
- added C35: 0.1uF, resistor:C0402
- added IC6: MUN3CAD01-SB, SamacSys_Parts:MUN3CAD01SB
- added IC7: FAN48610BUC50X, SamacSys_Parts:BGA9C40P3X3_122X122X62
- added R10: 12k, resistor:R0402
- added R16: 200k, resistor:R0402
- C1: value 2.2uF -> 22uF; device resistor:C0402 -> resistor:C0603
- C11, C14, C15, C2, C3, C39, C47: value 0.1uF -> 22uF; device resistor:C0402 -> resistor:C0603
- C16, C23, C26, C27, C8: value 22uF -> 0.1uF; device resistor:C0603 -> resistor:C0402
- C17, C18, C19, C36: value 22uF -> F930J107KBA; device resistor:C0603 -> SamacSys_Parts:CAPPM3528X210N
- C24: value 22uF -> 1uF; device resistor:C0603 -> resistor:C0402
- C25: value 22uF -> 2.2uF; device resistor:C0603 -> resistor:C0402
- C37: value 2.2uF -> F930J107KBA; device resistor:C0402 -> SamacSys_Parts:CAPPM3528X210N
- C38: value 0.1uF -> F930J107KBA; device resistor:C0402 -> SamacSys_Parts:CAPPM3528X210N
- C4: value 1uF -> 0.1uF
- C40: value 1uF -> 22uF; device resistor:C0402 -> resistor:C0603
- C41, C42, C43: value F930J107KBA -> 22uF; device SamacSys_Parts:CAPPM3528X210N -> resistor:C0603
- C5: value F930J107KBA -> 1uF; device SamacSys_Parts:CAPPM3528X210N -> resistor:C0402
- C6: value F930J107KBA -> 2.2uF; device SamacSys_Parts:CAPPM3528X210N -> resistor:C0402
- C7: value F930J107KBA -> 0.1uF; device SamacSys_Parts:CAPPM3528X210N -> resistor:C0402
- IC1: value SIC431AED-T1-GE3 -> SiC431CED-T1-GE3
- IC2: value MUN3CAD01-SB -> SiC431CED-T1-GE3; device SamacSys_Parts:MUN3CAD01SB -> personal:SIC431AEDT1GE3
- IC3: value SIC431AED-T1-GE3 -> TPS63810YFFR; device personal:SIC431AEDT1GE3 -> SamacSys_Parts:BGA15C40P3X5_134X226X62
- IC4: value MUN3CAD01-SB -> MUN3CAD03-SE; device SamacSys_Parts:MUN3CAD01SB -> SamacSys_Parts:MUN3CAD03SE
- IC5: value FAN48610BUC50X -> MUN3CAD01-SB; device SamacSys_Parts:BGA9C40P3X3_122X122X62 -> SamacSys_Parts:MUN3CAD01SB
- L1: value 1286AS-H-R47M=P2 -> MPXV1D0840L1R0; device SamacSys_Parts:1286ASH1R0MP2 -> SamacSys_Parts:INDPM8680X400N
- L3: value MPXV1D0840L1R0 -> TFM201208BLE-R47MTCF; device SamacSys_Parts:INDPM8680X400N -> Inductor:INDC2009X120
- L4: value TFM201208BLE-R47MTCF -> 1286AS-H-R47M=P2; device Inductor:INDC2009X120 -> SamacSys_Parts:1286ASH1R0MP2
- R11: value 100k -> 200k
- R12: value 11k -> 133k
- R13: value 12k -> 200k
- R14, R15: value 510k -> 187k
- R2: value 6.67k -> 510k
- R3: value 10K -> 510k
- R4: value 11k -> 6.67k
- R5: value 12k -> 10K
- R6: value 11k -> 100k
- R9: value 12k -> 11k
- moved C48 33.6 mm to (25.8, 0.13), flipped to the top, turned to 90 degrees
- moved C36 28.2 mm to (-4.08, 16.6), turned to 270 degrees
- moved C14 25.6 mm to (19.9, 16.5), flipped to the bottom, turned to 270 degrees
- moved C18 25.4 mm to (18.0, 16.5), turned to 270 degrees
- moved C16 25.2 mm to (13.2, 13.2), turned to 0 degrees
- moved TP1 25.1 mm to (-1.52, -2.54)
- moved TP4 25.1 mm to (23.6, -2.41)
- moved C29 24.7 mm to (-4.77, 16.5)
- moved C17 23.8 mm to (14.6, 16.5), turned to 270 degrees
- moved C23 23.6 mm to (4.73, 10.9), turned to 135 degrees
- moved C30 23.5 mm to (-2.37, 16.5)
- moved C27 23.1 mm to (-5.50, 14.2), turned to 0 degrees
- moved C28 22.3 mm to (-3.57, 16.5)
- moved R6 20.7 mm to (8.03, 9.21), turned to 270 degrees
- moved C50 20.0 mm to (3.74, -2.54), flipped to the top, turned to 0 degrees
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- renumbered C51 to C31, C52 to C32, C53 to C33, C54 to C34
Connections:
- net +5V: now also C24.1, C25.1, C5.1, C50.1, C6.1, IC2.12, IC2.15, IC7.A1, IC7.A2; no longer C1.1, C26.1, C37.1, C4.1, C40.1, IC3.12, IC3.15, IC5.A1, IC5.A2
- net 1.15V: now also C27.2, C28.1, C29.1, C30.1, C35.1, C36.1, C37.1, C38.1, IC2.18, L2.2, R9.2; no longer C14.1, C39.2, C41.1, C42.1, C43.1, C48.1, C49.1, C50.1, IC3.18, L3.2, R12.2
- net 1.1V: now also C48.1, IC6.8, R15.2, TP4.TP; no longer C23.1, IC4.8, R6.2, TP1.TP
- net 1.25V: now also C47.1, IC5.8, R13.2, TP3.TP; no longer C36.1, IC2.8, R19.2, TP2.TP
- net 1.5V: now also C43.1, C44.1, IC4.8, R11.2, TP2.TP; no longer C19.1, C21.1, PS2.8, R4.2, TP3.TP
- net 1V: now also C10.1, C11.1, C14.1, C16.1, C17.1, C18.1, C19.1, C8.2, C9.1, L1.2, R4.2; no longer C20.1, C27.1, C28.1, C29.1, C3.2, C30.1, C5.1, C6.1, C7.1, L2.2, R2.2
- net 3.3V: now also C40.1, C41.1, IC3.E2, IC3.E3, TP1.TP; no longer C17.1, C18.1, PS1.E2, PS1.E3, TP4.TP
- net BOOT: now also C7.1; no longer C2.1
- net BOOT2: now also C26.1, IC2.23; no longer C38.1, IC3.23
- net FB: now also R4.1, R5.2; no longer R2.1, R3.2
- net FB1: now also IC4.7, R11.1, R12.2; no longer PS2.7, R4.1, R5.2
- net FB2: now also IC2.17, R10.2, R9.1; no longer IC3.17, R12.1, R13.2
- net GND: now also C2.2, C27.1, C3.2, C35.2, C38.2, C39.2, C8.1, IC2.13, IC2.16, IC2.25, IC2.27, IC2.29, IC2.3, IC2.4, IC3.B1, IC3.C1, IC3.C2, IC3.C3, IC4.5, IC4.9, IC5.2, IC5.6, IC6.2, IC6.6, IC7.C1, IC7.C2, IC7.C3, R10.1, R12.1, R16.1, R2.1; no longer C26.2, C27.2, C3.1, C39.1, C56.2, C7.2, C8.2, IC2.2, IC2.6, IC3.13, IC3.16, IC3.25, IC3.27, IC3.29, IC3.3, IC3.4, IC4.2, IC5.C1, IC5.C2, IC5.C3, PS1.B1, PS1.C1, PS1.C2, PS1.C3, PS2.5, PS2.6, PS2.9, R13.1, R15.1, R20.1, R9.1
- net N$1: now also IC6.3, R15.1, R16.2; no longer IC4.3, R6.1, R9.2
- net N$12: now also IC2.19, R6.1; no longer IC3.19, R11.1
- net N$13: now also IC2.5, IC2.6, IC2.7, IC2.8, IC2.9, L2.1; no longer IC3.5, IC3.6, IC3.7, IC3.8, IC3.9, L3.1
- net N$14: now also IC2.21, R7.2; no longer IC3.21, R14.2
- net N$15: now also IC2.20, R8.2; no longer IC3.20, R15.2
- net N$2: now also IC5.3, R13.1, R14.2; no longer IC2.3, R19.1, R20.2
- net N$6: now also R2.2; no longer R7.2
- net N$7: now also L1.1; no longer L2.1
- net N$8: now also R3.2; no longer R8.2
- net PHASE: now also C7.2; no longer C2.2
- net PHASE2: now also C26.2, IC2.24; no longer C38.2, IC3.24
- net SW: now also IC7.B1, IC7.B2, L4.2; no longer IC5.B1, IC5.B2, L1.2
- net SW1: now also IC3.B2, IC3.B3, L3.1; no longer L4.1, PS1.B2, PS1.B3
- net SW2: now also IC3.D2, IC3.D3, L3.2; no longer L4.2, PS1.D2, PS1.D3
- net VIN: now also C1.1, C2.1, C20.1, C21.1, C23.1, C3.1, C39.1, C4.1, C42.1, C49.1, IC2.2, IC2.22, IC2.26, IC3.A1, IC3.A2, IC3.A3, IC4.3, IC4.4, IC5.1, IC5.7, IC6.1, IC6.7, IC7.A3, IC7.B3, L4.1, R6.2; no longer C10.1, C11.1, C16.1, C24.1, C25.1, C44.1, C47.1, C56.1, C8.1, C9.1, IC2.7, IC3.1, IC3.2, IC3.22, IC3.26, IC4.7, IC5.A3, IC5.B3, L1.1, PS1.A1, PS1.A2, PS1.A3, PS2.1, PS2.3, PS2.4, R11.2
