File: cafereg2.sch (EAGLE design)
At the start: 83 parts, among them IC1 SIC431AED-T1-GE3, IC2 MUN3CAD01-SB, IC3 SIC431AED-T1-GE3, IC4 MUN3CAD01-SB, IC5 FAN48610BUC50X

Commit message: update bom
Parts:
- removed C56: 22uF, resistor:C-USC0603
- removed PS1: TPS63810YFFR, SamacSys_Parts:TPS63810YFFR
- removed PS2: MUN3CAD03-SE, SamacSys_Parts:MUN3CAD03-SE
- removed R19: 11k, resistor:R-US_R0402
- removed R20: 12k, resistor:R-US_R0402
- added C35: 0.1uF, resistor:C-USC0402
- added IC6: MUN3CAD01-SB, SamacSys_Parts:MUN3CAD01-SB
- added IC7: FAN48610BUC50X, SamacSys_Parts:FAN48610BUC50X
- added R10: 12k, resistor:R-US_R0402
- added R16: 200k, resistor:R-US_R0402
- C1: value 2.2uF -> 22uF; device resistor:C-USC0402 -> resistor:C-USC0603
- C11, C14, C15, C2, C3, C39, C47: value 0.1uF -> 22uF; device resistor:C-USC0402 -> resistor:C-USC0603
- C16, C23, C26, C27, C8: value 22uF -> 0.1uF; device resistor:C-USC0603 -> resistor:C-USC0402
- C17, C18, C19, C36: value 22uF -> F930J107KBA; device resistor:C-USC0603 -> SamacSys_Parts:F930J107KBA
- C24: value 22uF -> 1uF; device resistor:C-USC0603 -> resistor:C-USC0402
- C25: value 22uF -> 2.2uF; device resistor:C-USC0603 -> resistor:C-USC0402
- C37: value 2.2uF -> F930J107KBA; device resistor:C-USC0402 -> SamacSys_Parts:F930J107KBA
- C38: value 0.1uF -> F930J107KBA; device resistor:C-USC0402 -> SamacSys_Parts:F930J107KBA
- C4: value 1uF -> 0.1uF
- C40: value 1uF -> 22uF; device resistor:C-USC0402 -> resistor:C-USC0603
- C41, C42, C43: value F930J107KBA -> 22uF; device SamacSys_Parts:F930J107KBA -> resistor:C-USC0603
- C5: value F930J107KBA -> 1uF; device SamacSys_Parts:F930J107KBA -> resistor:C-USC0402
- C6: value F930J107KBA -> 2.2uF; device SamacSys_Parts:F930J107KBA -> resistor:C-USC0402
- C7: value F930J107KBA -> 0.1uF; device SamacSys_Parts:F930J107KBA -> resistor:C-USC0402
- IC1: value SIC431AED-T1-GE3 -> SiC431CED-T1-GE3
- IC2: value MUN3CAD01-SB -> SiC431CED-T1-GE3; device SamacSys_Parts:MUN3CAD01-SB -> personal:SIC431AED-T1-GE3
- IC3: value SIC431AED-T1-GE3 -> TPS63810YFFR; device personal:SIC431AED-T1-GE3 -> SamacSys_Parts:TPS63810YFFR
- IC4: value MUN3CAD01-SB -> MUN3CAD03-SE; device SamacSys_Parts:MUN3CAD01-SB -> SamacSys_Parts:MUN3CAD03-SE
- IC5: value FAN48610BUC50X -> MUN3CAD01-SB; device SamacSys_Parts:FAN48610BUC50X -> SamacSys_Parts:MUN3CAD01-SB
- L1: value 1286AS-H-R47M=P2 -> MPXV1D0840L1R0; device SamacSys_Parts:1286AS-H-R47M=P2 -> SamacSys_Parts:MPXV1D0840L1R0
- L3: value MPXV1D0840L1R0 -> TFM201208BLE-R47MTCF; device SamacSys_Parts:MPXV1D0840L1R0 -> Inductor:L_CHIP-0805(2012-METRIC)
- L4: value TFM201208BLE-R47MTCF -> 1286AS-H-R47M=P2; device Inductor:L_CHIP-0805(2012-METRIC) -> SamacSys_Parts:1286AS-H-R47M=P2
- R11: value 100k -> 200k
- R12: value 11k -> 133k
- R13: value 12k -> 200k
- R14, R15: value 510k -> 187k
- R2: value 6.67k -> 510k
- R3: value 10K -> 510k
- R4: value 11k -> 6.67k
- R5: value 12k -> 10K
- R6: value 11k -> 100k
- R9: value 12k -> 11k
- renumbered C51 to C31, C52 to C32, C53 to C33, C54 to C34
Connections:
- net +5V: now also C24.1, C25.1, C5.1, C50.1, C6.1, IC2.VDD, IC2.VDRV, IC7.VOUT_1, IC7.VOUT_2; no longer C1.1, C26.1, C37.1, C4.1, C40.1, IC3.VDD, IC3.VDRV, IC5.VOUT_1, IC5.VOUT_2
- net 1.15V: now also C27.2, C28.1, C29.1, C30.1, C35.1, C36.+, C37.+, C38.+, IC2.VOUT, L2.2, R9.2; no longer C14.1, C39.2, C41.+, C42.+, C43.+, C48.1, C49.1, C50.1, IC3.VOUT, L3.2, R12.2
- net 1.1V: now also C48.1, IC6.VOUT, R15.2, TP4.TP; no longer C23.1, IC4.VOUT, R6.2, TP1.TP
- net 1.25V: now also C47.1, IC5.VOUT, R13.2, TP3.TP; no longer C36.1, IC2.VOUT, R19.2, TP2.TP
- net 1.5V: now also C43.1, C44.1, IC4.VOUT, R11.2, TP2.TP; no longer C19.1, C21.1, PS2.VOUT, R4.2, TP3.TP
- net 1V: now also C10.1, C11.1, C14.1, C16.1, C17.+, C18.+, C19.+, C8.2, C9.1, L1.2, R4.2; no longer C20.1, C27.1, C28.1, C29.1, C3.2, C30.1, C5.+, C6.+, C7.+, L2.2, R2.2
- net 3.3V: now also C40.1, C41.1, IC3.VOUT_1, IC3.VOUT_2, TP1.TP; no longer C17.1, C18.1, PS1.VOUT_1, PS1.VOUT_2, TP4.TP
- net BOOT: now also C7.1; no longer C2.1
- net BOOT2: now also C26.1, IC2.BOOT; no longer C38.1, IC3.BOOT
- net FB: now also R4.1, R5.2; no longer R2.1, R3.2
- net FB1: now also IC4.FB, R11.1, R12.2; no longer PS2.FB, R4.1, R5.2
- net FB2: now also IC2.FB, R10.2, R9.1; no longer IC3.FB, R12.1, R13.2
- net GND: now also C17.-, C18.-, C19.-, C2.2, C27.1, C3.2, C35.2, C36.-, C37.-, C38.-, C39.2, C41.2, C42.2, C43.2, C5.2, C6.2, C8.1, IC2.AGND_1, IC2.AGND_2, IC2.PGND_1, IC2.PGND_2, IC2.PGND_3, IC2.PGND_4, IC3.AGND, IC3.GND_1, IC3.GND_2, IC3.VSEL, IC4.GND_3, IC5.GND_1, IC5.GND_2, IC6.GND_1, IC6.GND_2, IC7.AGND, IC7.PGND_1, IC7.PGND_2, R10.1, R12.1, R16.1, R2.1; no longer C17.2, C18.2, C19.2, C26.2, C27.2, C3.1, C36.2, C37.2, C39.1, C41.-, C42.-, C43.-, C5.-, C56.2, C6.-, C7.-, C8.2, IC2.GND_1, IC2.GND_2, IC3.AGND_1, IC3.AGND_2, IC3.PGND_1, IC3.PGND_2, IC3.PGND_3, IC3.PGND_4, IC5.AGND, IC5.PGND_1, IC5.PGND_2, PS1.AGND, PS1.GND_1, PS1.GND_2, PS1.VSEL, PS2.GND_1, PS2.GND_2, PS2.GND_3, R13.1, R15.1, R20.1, R9.1
- net N$1: now also IC6.FB, R15.1, R16.2; no longer IC4.FB, R6.1, R9.2
- net N$12: now also IC2.EN, R6.1; no longer IC3.EN, R11.1
- net N$13: now also IC2.SW_1, IC2.SW_2, IC2.SW_3, IC2.SW_4, IC2.SW_5, L2.1; no longer IC3.SW_1, IC3.SW_2, IC3.SW_3, IC3.SW_4, IC3.SW_5, L3.1
- net N$14: now also IC2.MODE1, R7.2; no longer IC3.MODE1, R14.2
- net N$15: now also IC2.MODE2, R8.2; no longer IC3.MODE2, R15.2
- net N$2: now also IC5.FB, R13.1, R14.2; no longer IC2.FB, R19.1, R20.2
- net N$6: now also R2.2; no longer R7.2
- net N$7: now also L1.1; no longer L2.1
- net N$8: now also R3.2; no longer R8.2
- net PHASE: now also C7.2; no longer C2.2
- net PHASE2: now also C26.2, IC2.PHASE; no longer C38.2, IC3.PHASE
- net SW: now also IC7.SW_1, IC7.SW_2, L4.2; no longer IC5.SW_1, IC5.SW_2, L1.2
- net SW1: now also IC3.LX1_1, IC3.LX1_2, L3.1; no longer L4.1, PS1.LX1_1, PS1.LX1_2
- net SW2: now also IC3.LX2_1, IC3.LX2_2, L3.2; no longer L4.2, PS1.LX2_1, PS1.LX2_2
- net VIN: now also C1.1, C2.1, C20.1, C21.1, C23.1, C3.1, C39.1, C4.1, C42.1, C49.1, IC2.VIN_1, IC2.VIN_2, IC2.VIN_3, IC2.VIN_4, IC3.EN, IC4.VIN_1, IC4.VIN_2, IC6.EN, IC6.VIN, IC7.EN, IC7.VIN, L4.1, R6.2; no longer C10.1, C11.1, C16.1, C24.1, C25.1, C44.1, C47.1, C56.1, C8.1, C9.1, IC2.EN, IC2.VIN, IC3.VIN_3, IC3.VIN_4, IC4.VIN, L1.1, PS1.EN, PS1.VIN_1, PS1.VIN_2, PS2.EN, PS2.VIN_1, PS2.VIN_2, R11.2
Other:
- note added: "(1.161V nom)"
- note added: "(1.242V nom)"
